File: KiCad/slime_tracker.kicad_pcb (KiCad board)
At the start: 2 copper layers, 80.2 x 32 mm, 51 parts, among them J1 batt, J2 Extension, J3 USB_C_Receptacle_PowerOnly_6P, SW1 SW_DPDT_x2, U1 TP4056, U3 TPS7A0333PDBVR, U4 ESP32 SUPER MINI C3, U5 TPS61090

Commit message: Rev_02
Parts:
- removed R12: 10kΩ, Resistor_SMD:R_0603_1608Metric
- R11: value 2kΩ -> 3kΩ
- moved J1 5.01 mm to (75.8, 60.1)
- moved C1 0.25 mm to (133.2, 73.8)
- moved C6 0.25 mm to (130.5, 73.8)
Connections:
- U1 pad 1: Net-(D1-A) -> unconnected-(U1-NC-Pad1)
- U5 pad 17: (no net) -> BAT-
Routing:
- net BAT-: track 25.9 -> 6.80 mm, vias 192 -> 186
- net Net-(D1-A): track 34.7 -> 28.5 mm
- net BAT+: track 12.4 -> 14.1 mm
- net Net-(U1-!CHRG): track 8.48 -> 7.16 mm
- net Net-(U1-!STDBY): track 12.1 -> 11.3 mm
